File: kicad_project/temp_sensor.sch (KiCad schematic (older format))
At the start: 37 parts, among them J1 Battery port, J10 MOSI, J11 SCLK, J12 IO14, J13 IO12, J14 IO2, J15 flash, J16 SDA, J17 SCL, J2 USB_B_Micro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

Commit message: Updated project files and gerber data
Parts:
- removed C2: 100uF, Capacitor_SMD:C_0805_2012Metric_Pad1.15x1.40mm_HandSolder, symbol Device:C
- removed C3: 1uF, Capacitor_SMD:C_0805_2012Metric_Pad1.15x1.40mm_HandSolder, symbol Device:C
- removed D1: S2, LED_SMD:LED_0805_2012Metric_Pad1.15x1.40mm_HandSolder, symbol Device:LED
- removed D2: S1, LED_SMD:LED_0805_2012Metric_Pad1.15x1.40mm_HandSolder, symbol Device:LED
- removed J1: Battery port, Connector_PinHeader_2.54mm:PinHeader_1x02_P2.54mm_Vertical, symbol Connector:Conn_01x02_Male
- removed J11: SCLK, TestPoint:TestPoint_Pad_D1.5mm, symbol Connector:Conn_01x01_Female
- removed J12: IO14, TestPoint:TestPoint_Pad_D1.5mm, symbol Connector:Conn_01x01_Female
- removed J13: IO12, TestPoint:TestPoint_Pad_D1.5mm, symbol Connector:Conn_01x01_Female
- removed J14: IO2, TestPoint:TestPoint_Pad_D1.5mm, symbol Connector:Conn_01x01_Female
- removed J15: flash, Connector_PinHeader_2.54mm:PinHeader_1x02_P2.54mm_Vertical, symbol Connector:Conn_01x02_Male
- removed J2: USB_B_Micro, Connector_USB:USB_Micro-B_Molex-105017-0001, symbol Connector:USB_B_Micro
- removed J3: Flashing, Connector_PinHeader_2.54mm:PinHeader_1x04_P2.54mm_Vertical, symbol Connector:Conn_01x04_Male
- removed J5: reset, Connector_PinHeader_2.54mm:PinHeader_1x02_P2.54mm_Vertical, symbol Connector:Conn_01x02_Male
- removed R3: 470R, Resistor_SMD:R_0805_2012Metric_Pad1.15x1.40mm_HandSolder, symbol Device:R
- removed R4, R5: 10k, Resistor_SMD:R_0805_2012Metric_Pad1.15x1.40mm_HandSolder, symbol Device:R
- removed U2: MCP9808_MSOP, Package_SO:MSOP-8_3x3mm_P0.65mm, symbol Sensor_Temperature:MCP9804_MSOP
- removed U3: MCP73833, Package_SO:MSOP-10_3x3mm_P0.5mm, symbol CustomComponents:MCP73833
- removed U4: TC1262-33, Package_TO_SOT_SMD:SOT-223-3_TabPin2, symbol Regulator_Linear:TC1262-33
- added C5: 4.7-22 uF, Capacitor_SMD:C_0805_2012Metric_Pad1.15x1.40mm_HandSolder, symbol Device:C
- added F1: Polyfuse, Fuse:Fuse_0603_1608Metric_Pad1.05x0.95mm_HandSolder, symbol Device:Polyfuse
- added IC1: STM1061, Package_TO_SOT_SMD:SOT-23, symbol opendous:STM1061
- added IO1: GPIO14, TestPoint:TestPoint_Pad_D1.5mm, symbol Connector:Conn_01x01_Female
- added IO3: ADC, TestPoint:TestPoint_Pad_D1.5mm, symbol Connector:Conn_01x01_Female
- added J1: BAT+, TestPoint:TestPoint_Pad_2.5x2.5mm, symbol Connector:Conn_01x01_Female
- added J2: 3V3, TestPoint:TestPoint_Pad_D1.5mm, symbol Connector:Conn_01x01_Female
- added J3: GND, TestPoint:TestPoint_Pad_D1.5mm, symbol Connector:Conn_01x01_Female
- added L1: 4.7 uH, Inductor_SMD:L_0805_2012Metric_Pad1.15x1.40mm_HandSolder, symbol Device:L
- added SW1: SW_reset, Button_Switch_SMD:SW_SPST_Panasonic_EVQPL_3PL_5PL_PT_A08, symbol Switch:SW_Push
- added SW2: SW_flash, Button_Switch_SMD:SW_SPST_Panasonic_EVQPL_3PL_5PL_PT_A08, symbol Switch:SW_Push
- added U2: MCP1603T-330I_OS, Package_TO_SOT_SMD:TSOT-23-5_HandSoldering, symbol temp_sensor-rescue:MCP1603T-330I_OS-MCP1603T-330I_OS
- added U4: SHT31-DIS-B, SHT31-DIS-B:SON50P250X250X100-9N, symbol temp_sensor-rescue:SHT31-DIS-B-SHT31-DIS-B
- C1: value 1uF -> 100uF; footprint Capacitor_SMD:C_0805_2012Metric_Pad1.15x1.40mm_HandSolder -> Capacitor_SMD:CP_Elec_5x5.3
- C4: value 330uF -> 200 uF; footprint Capacitor_SMD:CP_Elec_6.3x9.9 -> Capacitor_SMD:CP_Elec_5x5.3
- IO2: renamed from IO13; value pad -> GPIO12
- J10: value MOSI -> GND
- J6: value CSO -> BAT-; footprint TestPoint:TestPoint_Pad_D1.5mm -> TestPoint:TestPoint_Pad_2.5x2.5mm
- J7: value MISO -> TX
- J8: value IO9 -> RX
- J9: value IO10 -> 3V3
- R2: value 470R -> 10k
- R6: value 330k -> 4k7
- R7: value 100k -> 4k7
- U1: symbol ESP8266:ESP-12E -> temp_sensor-rescue:ESP-12E-ESP8266
- renumbered J16 to J4, J17 to J5, R8 to R1, R9 to R5, R10 to R8, R11 to R9
Connections:
- net labels added: GND
- net labels removed: +5V
- wire segments 101 -> 106
- no-connect marks 10 -> 9
